Commit message: quad.xacro: Add own quadrotor defns
Add our own quadrotor definitions in the xacro rather than just including
a preexisting launch file. Makes it easier to modify

File: rl_env/src/Env/HectorQuad/quad.gazebo.xacro (robot description, xacro)
@@ -1,5 +1,43 @@
 <?xml version="1.0"?>
 <robot name="quadrotor" xmlns:xacro="http://ros.org/wiki/xacro">
-    <xacro:include filename="$(find hector_quadrotor_description)/urdf/quadrotor.urdf.xacro" />
-    <xacro:include filename="$(find hector_quadrotor_gazebo)/urdf/quadrotor_plugins.gazebo.xacro" />
+  <!-- Taken fromthe Xacro file : <xacro:include filename="$(find hector_quadrotor_description)/urdf/quadrotor.urdf.xacro" /> -->
+  <xacro:property name="pi" value="3.1415926535897931" />
+  <!-- Sonar sensor include -->
+  <!-- <xacro:include filename="$(find hector_sensors_description)/urdf/sonar_sensor.urdf.xacro" /> -->
+  <!-- Main quadrotor link -->
+  <link name="base_link">
+    <inertial>
+      <mass value="1.477" />
+      <origin xyz="0 0 0" />
+      <inertia ixx="0.01152" ixy="0.0" ixz="0.0" iyy="0.01152" iyz="0.0" izz="0.0218" />
+    </inertial>
+    <visual>
+      <origin xyz="0 0 0" rpy="0 0 0" />
+      <geometry>
+        <mesh filename="package://hector_quadrotor_description/meshes/quadrotor/quadrotor_base.dae"/>
+      </geometry>
+    </visual>
+    <collision>
+      <origin xyz="0 0 0" rpy="0 0 0" />
+      <geometry>
+        <mesh filename="package://hector_quadrotor_description/meshes/quadrotor/quadrotor_base.stl"/>
+      </geometry>
+    </collision>
+  </link>
+  <!-- Sonar height sensor -->
+  <!-- <xacro:sonar_sensor name="sonar" parent="base_link" ros_topic="sonar_height" update_rate="10" min_range="0.03" max_range="3.0" field_of_view="${40*pi/180}" ray_count="3">
+    <origin xyz="-0.16 0.0 -0.012" rpy="0 ${90*pi/180} 0"/>
+  </xacro:sonar_sensor> -->
+  <!-- Taken from the Xacro file : <xacro:include filename="$(find hector_quadrotor_gazebo)/urdf/quadrotor_plugins.gazebo.xacro" /> -->
+  <arg name="world_frame" default="world"/> <!-- This should actually be "/world". See https://github.com/ros-simulation/gazebo_ros_pkgs/pull/324 -->
+  <arg name="base_link_frame" default="base_link"/>
+  <xacro:include filename="$(find hector_quadrotor_gazebo)/urdf/quadrotor_sensors.gazebo.xacro" />
+  <xacro:include filename="$(find hector_quadrotor_gazebo)/urdf/quadrotor_controller.gazebo.xacro" />
+  <xacro:include filename="$(find hector_quadrotor_gazebo)/urdf/quadrotor_propulsion.gazebo.xacro" />
+  <xacro:include filename="$(find hector_quadrotor_gazebo)/urdf/quadrotor_aerodynamics.gazebo.xacro" />
+  <!-- Quadrotor Gazebo Plugins -->
+  <xacro:quadrotor_sensors />
+  <xacro:quadrotor_controller />
+  <xacro:quadrotor_propulsion />
+  <xacro:quadrotor_aerodynamics />
 </robot>

Commit message: Added payload for quadrotor

File: rl_env/src/Env/HectorQuad/quad.gazebo.xacro (robot description, xacro)
@@ -25,4 +25,30 @@
     </collision>
   </link>
+  <link name="payload">
+    <visual>
+      <origin xyz="0 0 -1" rpy="0 0 0" />
+      <geometry>
+        <sphere radius="0.2"/>
+      </geometry>
+      <material name="blue">
+        <color rgba="0 0 .8 1"/>
+      </material>
+    </visual>
+    <inertial>
+      <mass value="1" />
+      <origin xyz="0 0 -1" />
+      <inertia ixx="1" iyy="1" izz="1" ixy="0" iyz="0" ixz="0" />
+    </inertial>
+    <collision>
+      <origin xyz="0 0 -1" rpy="0 0 0" />
+      <geometry>
+        <sphere radius="0.2"/>
+      </geometry>
+    </collision>
+  </link>
+  <joint name="payload_connector" type="fixed">
+    <parent link="base_link"/>
+    <child link="payload"/>
+  </joint>
   <!-- Sonar height sensor -->
   <!-- <xacro:sonar_sensor name="sonar" parent="base_link" ros_topic="sonar_height" update_rate="10" min_range="0.03" max_range="3.0" field_of_view="${40*pi/180}" ray_count="3">

Commit message: INCOMPLETE Attempt to fix joints.
This commit is incomplete.

File: rl_env/src/Env/HectorQuad/quad.gazebo.xacro (robot description, xacro)
@@ -47,7 +47,9 @@
     </collision>
   </link>
-  <joint name="payload_connector" type="fixed">
+  <joint name="payload_connector" type="floating">
     <parent link="base_link"/>
     <child link="payload"/>
+    <origin xyz="0 0 0" />
+    <limit lower="-0.01" upper="0.01" velocity="0.01" effort="1000" />
   </joint>
   <!-- Sonar height sensor -->

Commit message: Added payload based control

File: rl_env/src/Env/HectorQuad/quad.gazebo.xacro (robot description, xacro)
@@ -9,5 +9,5 @@
     <inertial>
       <mass value="1.477" />
-      <origin xyz="0 0 0" />
+      <origin xyz="0 0 0" rpy="0 0 0" />
       <inertia ixx="0.01152" ixy="0.0" ixz="0.0" iyy="0.01152" iyz="0.0" izz="0.0218" />
     </inertial>
@@ -27,29 +27,30 @@
   <link name="payload">
     <visual>
-      <origin xyz="0 0 -1" rpy="0 0 0" />
       <geometry>
-        <sphere radius="0.2"/>
+        <box size="0.6 0.6 0.6"/>
       </geometry>
       <material name="blue">
         <color rgba="0 0 .8 1"/>
       </material>
+      <origin xyz="0 0 0" rpy="0 0 0"/>
     </visual>
     <inertial>
-      <mass value="1" />
-      <origin xyz="0 0 -1" />
-      <inertia ixx="1" iyy="1" izz="1" ixy="0" iyz="0" ixz="0" />
+      <mass value="0.01" />
+      <inertia ixx="0.0006" iyy="0.0006" izz="0.0006" ixy="0" ixz="0" iyz="0" />
+      <origin rpy="0 0 0" xyz="0 0 0"/>
     </inertial>
     <collision>
-      <origin xyz="0 0 -1" rpy="0 0 0" />
+      <origin rpy="0 0 0" xyz="0 0 0"/>
       <geometry>
-        <sphere radius="0.2"/>
+        <box size="0.6 0.6 0.6"/>
       </geometry>
     </collision>
   </link>
-  <joint name="payload_connector" type="floating">
+  <joint name="payload_connector" type="revolute">
+    <origin xyz="0 0 -1" rpy="0 0 0" />
+    <axis xyz="0 0 1"/>
     <parent link="base_link"/>
     <child link="payload"/>
-    <origin xyz="0 0 0" />
-    <limit lower="-0.01" upper="0.01" velocity="0.01" effort="1000" />
+    <limit lower="-3.14" upper="3.14" effort="1000" velocity="1" />
   </joint>
   <!-- Sonar height sensor -->

Commit message: Added proper payload for control

File: rl_env/src/Env/HectorQuad/quad.gazebo.xacro (robot description, xacro)
@@ -28,14 +28,14 @@
     <visual>
       <geometry>
-        <box size="0.6 0.6 0.6"/>
+        <box size="0.3 0.3 0.3"/>
       </geometry>
       <material name="blue">
-        <color rgba="0 0 .8 1"/>
+        <color rgba="0 0.3 0 1"/>
       </material>
       <origin xyz="0 0 0" rpy="0 0 0"/>
     </visual>
     <inertial>
-      <mass value="0.01" />
-      <inertia ixx="0.0006" iyy="0.0006" izz="0.0006" ixy="0" ixz="0" iyz="0" />
+      <mass value="0.1" />
+      <inertia ixx="0.0015" iyy="0.0015" izz="0.0015" ixy="0" ixz="0" iyz="0" />
       <origin rpy="0 0 0" xyz="0 0 0"/>
     </inertial>
@@ -43,14 +43,14 @@
       <origin rpy="0 0 0" xyz="0 0 0"/>
       <geometry>
-        <box size="0.6 0.6 0.6"/>
+        <box size="0.3 0.3 0.3"/>
       </geometry>
     </collision>
   </link>
   <joint name="payload_connector" type="revolute">
-    <origin xyz="0 0 -1" rpy="0 0 0" />
+    <origin xyz="0 0 -0.3" rpy="0 0 0" />
     <axis xyz="0 0 1"/>
     <parent link="base_link"/>
     <child link="payload"/>
-    <limit lower="-3.14" upper="3.14" effort="1000" velocity="1" />
+    <limit lower="-0.01" upper="0.01" effort="1000" velocity="1" />
   </joint>
   <!-- Sonar height sensor -->

Commit message: Added trajectory control using waypoints and Pure Pursuit

File: rl_env/src/Env/HectorQuad/quad.gazebo.xacro (robot description, xacro)
@@ -33,13 +33,13 @@
         <color rgba="0 0.3 0 1"/>
       </material>
-      <origin xyz="0 0 0" rpy="0 0 0"/>
+      <origin xyz="0 0 -0.3" rpy="0 0 0"/>
     </visual>
     <inertial>
       <mass value="0.1" />
-      <inertia ixx="0.0015" iyy="0.0015" izz="0.0015" ixy="0" ixz="0" iyz="0" />
-      <origin rpy="0 0 0" xyz="0 0 0"/>
+      <inertia ixx="0.005" iyy="0.005" izz="0.005" ixy="0" ixz="0" iyz="0" />
+      <origin rpy="0 0 0" xyz="0 0 -0.3"/>
     </inertial>
     <collision>
-      <origin rpy="0 0 0" xyz="0 0 0"/>
+      <origin rpy="0 0 0" xyz="0 0 -0.3"/>
       <geometry>
         <box size="0.3 0.3 0.3"/>
@@ -48,9 +48,16 @@
   </link>
   <joint name="payload_connector" type="revolute">
-    <origin xyz="0 0 -0.3" rpy="0 0 0" />
-    <axis xyz="0 0 1"/>
+    <origin xyz="0 0 0" rpy="0 0 0" />
+    <axis xyz="1 0 0"/>
     <parent link="base_link"/>
     <child link="payload"/>
-    <limit lower="-0.01" upper="0.01" effort="1000" velocity="1" />
+    <limit lower="-1" upper="1" effort="1" velocity="1" />
+  </joint>
+<joint name="payload_connector2" type="revolute">
+    <origin xyz="0 0 0" rpy="0 0 0" />
+    <axis xyz="0 1 0"/>
+    <parent link="base_link"/>
+    <child link="payload"/>
+    <limit lower="-1" upper="1" effort="1" velocity="1" />
   </joint>
   <!-- Sonar height sensor -->

Commit message: rl_env: Add "use_payload" to toggle state

File: rl_env/src/Env/HectorQuad/quad.gazebo.xacro (robot description, xacro)
@@ -3,4 +3,5 @@
   <!-- Taken fromthe Xacro file : <xacro:include filename="$(find hector_quadrotor_description)/urdf/quadrotor.urdf.xacro" /> -->
   <xacro:property name="pi" value="3.1415926535897931" />
+  <xacro:arg name="use_payload" default="false" />
   <!-- Sonar sensor include -->
   <!-- <xacro:include filename="$(find hector_sensors_description)/urdf/sonar_sensor.urdf.xacro" /> -->
@@ -25,40 +26,42 @@
     </collision>
   </link>
-  <link name="payload">
-    <visual>
-      <geometry>
-        <box size="0.3 0.3 0.3"/>
-      </geometry>
-      <material name="blue">
-        <color rgba="0 0.3 0 1"/>
-      </material>
-      <origin xyz="0 0 -0.3" rpy="0 0 0"/>
-    </visual>
-    <inertial>
-      <mass value="0.1" />
-      <inertia ixx="0.005" iyy="0.005" izz="0.005" ixy="0" ixz="0" iyz="0" />
-      <origin rpy="0 0 0" xyz="0 0 -0.3"/>
-    </inertial>
-    <collision>
-      <origin rpy="0 0 0" xyz="0 0 -0.3"/>
-      <geometry>
-        <box size="0.3 0.3 0.3"/>
-      </geometry>
-    </collision>
-  </link>
-  <joint name="payload_connector" type="revolute">
-    <origin xyz="0 0 0" rpy="0 0 0" />
-    <axis xyz="1 0 0"/>
-    <parent link="base_link"/>
-    <child link="payload"/>
-    <limit lower="-1" upper="1" effort="1" velocity="1" />
-  </joint>
-<joint name="payload_connector2" type="revolute">
-    <origin xyz="0 0 0" rpy="0 0 0" />
-    <axis xyz="0 1 0"/>
-    <parent link="base_link"/>
-    <child link="payload"/>
-    <limit lower="-1" upper="1" effort="1" velocity="1" />
-  </joint>
+  <xacro:if value="$(arg use_payload)">
+    <link name="payload">
+      <visual>
+        <geometry>
+          <box size="0.3 0.3 0.3"/>
+        </geometry>
+        <material name="blue">
+          <color rgba="0 0.3 0 1"/>
+        </material>
+        <origin xyz="0 0 -0.3" rpy="0 0 0"/>
+      </visual>
+      <inertial>
+        <mass value="0.1" />
+        <inertia ixx="0.005" iyy="0.005" izz="0.005" ixy="0" ixz="0" iyz="0" />
+        <origin rpy="0 0 0" xyz="0 0 -0.3"/>
+      </inertial>
+      <collision>
+        <origin rpy="0 0 0" xyz="0 0 -0.3"/>
+        <geometry>
+          <box size="0.3 0.3 0.3"/>
+        </geometry>
+      </collision>
+    </link>
+    <joint name="payload_connector" type="revolute">
+      <origin xyz="0 0 0" rpy="0 0 0" />
+      <axis xyz="1 0 0"/>
+      <parent link="base_link"/>
+      <child link="payload"/>
+      <limit lower="-1" upper="1" effort="1" velocity="1" />
+    </joint>
+    <!-- <joint name="payload_connector2" type="revolute">
+      <origin xyz="0 0 0" rpy="0 0 0" />
+      <axis xyz="0 1 0"/>
+      <parent link="base_link"/>
+      <child link="payload"/>
+      <limit lower="-1" upper="1" effort="1" velocity="1" />
+    </joint> -->
+  </xacro:if>
   <!-- Sonar height sensor -->
   <!-- <xacro:sonar_sensor name="sonar" parent="base_link" ros_topic="sonar_height" update_rate="10" min_range="0.03" max_range="3.0" field_of_view="${40*pi/180}" ray_count="3">
@@ -68,9 +71,9 @@
   <arg name="world_frame" default="world"/> <!-- This should actually be "/world". See https://github.com/ros-simulation/gazebo_ros_pkgs/pull/324 -->
   <arg name="base_link_frame" default="base_link"/>
+  <!-- Quadrotor Gazebo Plugins -->
   <xacro:include filename="$(find hector_quadrotor_gazebo)/urdf/quadrotor_sensors.gazebo.xacro" />
   <xacro:include filename="$(find hector_quadrotor_gazebo)/urdf/quadrotor_controller.gazebo.xacro" />
   <xacro:include filename="$(find hector_quadrotor_gazebo)/urdf/quadrotor_propulsion.gazebo.xacro" />
   <xacro:include filename="$(find hector_quadrotor_gazebo)/urdf/quadrotor_aerodynamics.gazebo.xacro" />
-  <!-- Quadrotor Gazebo Plugins -->
   <xacro:quadrotor_sensors />
   <xacro:quadrotor_controller />

Commit message: world.cc: Simplify code and add debug statements

File: rl_env/src/Env/HectorQuad/quad.gazebo.xacro (robot description, xacro)
@@ -56,5 +56,5 @@
       <limit lower="-1" upper="1" effort="1" velocity="1" />
     </joint>
-    <!-- <joint name="payload_connector2" type="revolute">
+    <joint name="payload_connector2" type="revolute">
       <origin xyz="0 0 0" rpy="0 0 0" />
       <axis xyz="0 1 0"/>
@@ -62,5 +62,5 @@
       <child link="payload"/>
       <limit lower="-1" upper="1" effort="1" velocity="1" />
-    </joint> -->
+    </joint>
   </xacro:if>
   <!-- Sonar height sensor -->

Commit message: quad.gazebo.xacro: Use chain type joint

File: rl_env/src/Env/HectorQuad/quad.gazebo.xacro (robot description, xacro)
@@ -4,4 +4,15 @@
   <xacro:property name="pi" value="3.1415926535897931" />
   <xacro:arg name="use_payload" default="false" />
+  <!-- value for chain's mass -->
+  <xacro:property name="payload_mass" value="0.1" />
+  <!-- Cube dimensions (side x side x side) of payload -->
+  <xacro:property name="payload_side" value="0.3" />
+  <!-- value for chain's mass -->
+  <xacro:property name="chain_mass" value="0.001" />
+  <!-- Square dimensions (width x width) of links in the chain -->
+  <xacro:property name="chain_width" value="0.03" />
+  <xacro:property name="chain_height" value="0.3" />
+  <!-- Space btw top of beam and the each joint -->
+  <!-- <xacro:property name="chain_axel_offset" value="0.05" /> -->
   <!-- Sonar sensor include -->
   <!-- <xacro:include filename="$(find hector_sensors_description)/urdf/sonar_sensor.urdf.xacro" /> -->
@@ -27,40 +38,68 @@
   </link>
   <xacro:if value="$(arg use_payload)">
+    <joint name="joint1" type="revolute">
+      <parent link="base_link"/>
+      <child link="link1"/>
+      <origin xyz="0 0 0" rpy="0 0 0"/>
+      <axis xyz="0 1 0"/>
+      <limit upper="0.1" lower="-0.1" velocity="10" effort="1"/>
+    </joint>
+    <link name="link1">
+      <collision>
+        <origin xyz="0 0 ${-chain_height/2}" rpy="0 0 0"/>
+        <geometry>
+          <box size="${chain_width} ${chain_width} ${chain_height}"/>
+        </geometry>
+      </collision>
+      <visual>
+        <origin xyz="0 0 ${-chain_height/2}" rpy="0 0 0"/>
+        <geometry>
+          <box size="${chain_width} ${chain_width} ${chain_height}"/>
+        </geometry>
+        <material name="red">
+          <color rgba="1 0 0 1"/>
+        </material>
+      </visual>
+      <inertial>
+        <origin xyz="0 0 ${-chain_height/2}" rpy="0 0 0"/>
+        <mass value="${chain_mass}"/>
+        <inertia
+          ixx="${chain_mass / 12.0 * (chain_width*chain_width + chain_height*chain_height)}" ixy="0.0" ixz="0.0"
+          iyy="${chain_mass / 12.0 * (chain_height*chain_height + chain_width*chain_width)}" iyz="0.0"
+          izz="${chain_mass / 12.0 * (chain_width*chain_width + chain_width*chain_width)}"/>
+      </inertial>
+    </link>
+    <joint name="joint_payload" type="revolute">
+      <origin xyz="0 0 ${-chain_height}" rpy="0 0 0"/>
+      <axis xyz="0 1 0"/>
+      <parent link="link1"/>
+      <child link="payload"/>
+      <limit upper="0.1" lower="-0.1" velocity="10" effort="1"/>
+    </joint>
     <link name="payload">
       <visual>
         <geometry>
-          <box size="0.3 0.3 0.3"/>
+          <box size="${payload_side} ${payload_side} ${payload_side}"/>
         </geometry>
-        <material name="blue">
+        <material name="green">
           <color rgba="0 0.3 0 1"/>
         </material>
-        <origin xyz="0 0 -0.3" rpy="0 0 0"/>
+        <origin xyz="0 0 0" rpy="0 0 0"/>
       </visual>
       <inertial>
-        <mass value="0.1" />
-        <inertia ixx="0.005" iyy="0.005" izz="0.005" ixy="0" ixz="0" iyz="0" />
-        <origin rpy="0 0 0" xyz="0 0 -0.3"/>
+        <mass value="${payload_mass}" />
+        <inertia
+          ixx="${payload_mass / 12.0 * (payload_side*payload_side + payload_side*payload_side)}" ixy="0.0" ixz="0.0"
+          iyy="${payload_mass / 12.0 * (payload_side*payload_side + payload_side*payload_side)}" iyz="0.0"
+          izz="${payload_mass / 12.0 * (payload_side*payload_side + payload_side*payload_side)}"/>
+        <origin rpy="0 0 0" xyz="0 0 0"/>
       </inertial>
       <collision>
-        <origin rpy="0 0 0" xyz="0 0 -0.3"/>
+        <origin rpy="0 0 0" xyz="0 0 0"/>
         <geometry>
-          <box size="0.3 0.3 0.3"/>
+          <box size="${payload_side} ${payload_side} ${payload_side}"/>
         </geometry>
       </collision>
     </link>
-    <joint name="payload_connector" type="revolute">
-      <origin xyz="0 0 0" rpy="0 0 0" />
-      <axis xyz="1 0 0"/>
-      <parent link="base_link"/>
-      <child link="payload"/>
-      <limit lower="-1" upper="1" effort="1" velocity="1" />
-    </joint>
-    <joint name="payload_connector2" type="revolute">
-      <origin xyz="0 0 0" rpy="0 0 0" />
-      <axis xyz="0 1 0"/>
-      <parent link="base_link"/>
-      <child link="payload"/>
-      <limit lower="-1" upper="1" effort="1" velocity="1" />
-    </joint>
   </xacro:if>
   <!-- Sonar height sensor -->
